Commit message: 09082026

File: demo/robot-simulator/navigation-stack/config/robot.urdf (robot description, URDF)
Before this commit: robot rovera_pi5, 4 links, 3 joints
Joints:
- joint base_link_to_laser: origin xyz=0 0 0.07 rpy=0 0 0 -> xyz=-0.0046412 0 0.094079 rpy=0 0 0

Commit message: 12082026-1

File: demo/robot-simulator/navigation-stack/config/robot.urdf (robot description, URDF)
Before this commit: robot rovera_pi5, 4 links, 3 joints
Links:
- link base_link: geometry collision box size=0.40 0.36 0.10; visual box size=0.40 0.36 0.10

Commit message: 14082026-3

File: demo/robot-simulator/navigation-stack/config/robot.urdf (robot description, URDF)
Before this commit: robot rovera_pi5, 4 links, 3 joints
Links:
- link base_link: geometry collision box size=0.30 0.20 0.10; visual box size=0.30 0.20 0.10

Commit message: 03092026

File: demo/robot-simulator/navigation-stack/config/robot.urdf (robot description, URDF)
Before this commit: robot rovera_pi5, 4 links, 3 joints
Links:
- link base_link: geometry collision box size=0.30 0.20 0.15; visual box size=0.30 0.20 0.15
Joints:
- joint base_footprint_to_base_link: origin xyz=0 0 0.05 rpy=0 0 0 -> xyz=0 0 0.075 rpy=0 0 0
- joint base_link_to_laser: origin xyz=-0.0046412 0 0.094079 rpy=0 0 0 -> xyz=0 0 0.075 rpy=0 0 0

Commit message: 04092026-1

File: demo/robot-simulator/navigation-stack/config/robot.urdf (robot description, URDF)
Before this commit: robot rovera_pi5, 4 links, 3 joints
Links:
- link base_link: geometry collision box size=0.31 0.20 0.15; visual box size=0.31 0.20 0.15
